File: carte d’acquisition -2026-02-08_124430/thermocouple.kicad_sch (KiCad schematic)
At the start: 6 parts, among them U6 MAX31855SASA_T, U6 MC74HC4067ADWR2G, U7 MC74HC4067ADWR2G

Commit message: Update thermocouple.kicad_sch
Connections:
- net GND: now also U7.15 (*E), U7.16 (I15), U7.17 (I14), U7.18 (I13), U7.19 (I12), U7.20 (I11), U7.21 (I10)
Changed lines of the file:
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@@
 	(paper "A4")
+	(junction
+		(at 133.35 120.65)
+		(diameter 0)
+		(color 0 0 0 0)
+	)
+	(junction
+		(at 133.35 125.73)
+		(diameter 0)
+		(color 0 0 0 0)
+	)
+	(junction
+		(at 133.35 123.19)
+		(diameter 0)
+		(color 0 0 0 0)
+	)
+	(junction
+		(at 133.35 118.11)
+		(diameter 0)
+		(color 0 0 0 0)
+	)
 	(junction
 		(at 243.84 134.62)
@@
 		(color 0 0 0 0)
 	)
+	(junction
+		(at 133.35 128.27)
+		(diameter 0)
+		(color 0 0 0 0)
+	)
+	(junction
+		(at 133.35 130.81)
+		(diameter 0)
+		(color 0 0 0 0)
+	)
 	(wire
 		(pts
@@
 	(wire
 		(pts
+			(xy 133.35 128.27) (xy 133.35 130.81)
+		)
+		(stroke
+			(width 0)
+			(type default)
+		)
+	)
+	(wire
+		(pts
 			(xy 246.38 62.23) (xy 243.84 62.23)
 		)
@@
 	(wire
 		(pts
+			(xy 133.35 123.19) (xy 133.35 125.73)
+		)
+		(stroke
+			(width 0)
+			(type default)
+		)
+	)
+	(wire
+		(pts
 			(xy 55.88 123.19) (xy 67.31 123.19)
 		)
@@
 	(wire
 		(pts
+			(xy 144.78 124.46) (xy 144.78 118.11)
+		)
+		(stroke
+			(width 0)
+			(type default)
+		)
+	)
+	(wire
+		(pts
+			(xy 133.35 120.65) (xy 133.35 123.19)
+		)
+		(stroke
+			(width 0)
+			(type default)
+		)
+	)
+	(wire
+		(pts
 			(xy 146.05 58.42) (xy 133.35 58.42)
 		)
@@
 	(wire
 		(pts
+			(xy 133.35 118.11) (xy 144.78 118.11)
+		)
+		(stroke
+			(width 0)
+			(type default)
+		)
+	)
+	(wire
+		(pts
 			(xy 67.31 53.34) (xy 67.31 35.56)
 		)
@@
 	(wire
 		(pts
+			(xy 133.35 130.81) (xy 133.35 133.35)
+		)
+		(stroke
+			(width 0)
+			(type default)
+		)
+	)
+	(wire
+		(pts
+			(xy 133.35 125.73) (xy 133.35 128.27)
+		)
+		(stroke
+			(width 0)
+			(type default)
+		)
+	)
+	(wire
+		(pts
 			(xy 55.88 73.66) (xy 67.31 73.66)
 		)
@@
 		(pts
 			(xy 146.05 81.28) (xy 133.35 81.28)
+		)
+		(stroke
+			(width 0)
+			(type default)
+		)
+	)
+	(wire
+		(pts
+			(xy 133.35 118.11) (xy 133.35 120.65)
 		)
 		(stroke
@@
 					(unit 1)
 				)
+			)
+		)
+	)
+	(symbol
+		(lib_id "power:GND")
+		(at 144.78 124.46 0)
+		(unit 1)
+		(exclude_from_sim no)
+		(in_bom yes)
+		(on_board yes)
+		(dnp no)
+		(fields_autoplaced yes)
+		(property "Reference" "#PWR033"
+			(at 144.78 130.81 0)
+			(effects
+				(font
+					(size 1.27 1.27)
+				)
+				(hide yes)
+			)
+		)
+		(property "Value" "GND"
+			(at 144.78 129.54 0)
+			(effects
+				(font
+					(size 1.27 1.27)
+				)
+			)
+		)
+		(property "Footprint" ""
+			(at 144.78 124.46 0)
+			(effects
+				(font
+					(size 1.27 1.27)
+				)
+				(hide yes)
+			)
+		)
+		(property "Datasheet" ""
+			(at 144.78 124.46 0)
+			(effects
+				(font
+					(size 1.27 1.27)
+				)
+				(hide yes)
+			)
+		)
+		(property "Description" "Power symbol creates a global label with name \"GND\" , ground"
+			(at 144.78 124.46 0)
+			(effects
+				(font
+					(size 1.27 1.27)
+				)
+				(hide yes)
+			)
+		)
+		(pin "1"
+		)
+		(instances
+			(project "acquisition"
+				(path "/eaacffe0-ee57-428e-a37e-5655e0922ccc/4a2889f9-cbe2-4e8a-8334-287f8d92a54d"
+					(reference "#PWR033")
+					(unit 1)
+				)

Commit message: Update thermocouple.kicad_sch
Parts:
- removed U6: MC74HC4067ADWR2G, SOIC-24WB_ONS, symbol MC74HC4067ADWR2G:MC74HC4067ADWR2G
- added U8: MC74HC4067ADWR2G, footprints:SOIC-24WB_ONS, symbol MC74HC4067ADWR2G:MC74HC4067ADWR2G
- U7: footprint SOIC-24WB_ONS -> footprints:SOIC-24WB_ONS
Connections:
- net 3V3: now also U8.24 (VCC)
- net GND: now also U8.12 (GND), U8.15 (~{E}), U8.16 (I15), U8.17 (I14), U8.18 (I13), U8.19 (I12), U8.20 (I11), U8.21 (I10)
- net bits_commende_0: now also U7.10 (S0), U8.10 (S0); no longer U7.11 (S1)
- net bits_commende_1: now also U7.11 (S1), U8.11 (S1); no longer U7.10 (S0)
- net bits_commende_2: now also U8.14 (S2)
- net bits_commende_3: now also U8.13 (S3)
- net capteur_1+: now also U8.9 (I0)
- net capteur_10+: now also U8.22 (I9)
- net capteur_2+: now also U8.8 (I1)
- net capteur_3+: now also U8.7 (I2)
- net capteur_4+: now also U8.6 (I3)
- net capteur_5+: now also U8.5 (I4)
- net capteur_6+: now also U8.4 (I5)
- net capteur_7+: now also U8.3 (I6)
- net capteur_8+: now also U8.2 (I7)
- net capteur_9+: now also U8.23 (I8)
- net at U6.3 (T+): now also U8.1 (OUT)
Other:
- moved on the sheet: U6
