File: carte d’acquisition -2026-02-08_124430/microcontrolleur.kicad_sch (KiCad schematic)
At the start: 34 parts, among them SW1 CK_KMS2xxG, SW2 BOOT, U1 STM32H747IITx, Y1 Crystal, Y2 Crystal

Commit message: arthur net
Connections:
- net BC0: now reaches U1.156 (PG12)
- net BC2: now reaches U1.158 (PG14)
- net BC3: now reaches U1.161 (PG15)
- net I2C1_SCL: now reaches U1.165 (PB6)
- net I2C1_SDA: now reaches U1.166 (PB7)
- net SPI5_NSS: now reaches U1.26 (PF6)
- net SPI5_SCK: now reaches U1.27 (PF7)
- net SPI5_MISO: now reaches U1.28 (PF8)
- net SPI5_MOSI: now reaches U1.29 (PF9)
- net SPI4_NSS: now reaches U1.3 (PE4)
- net SPI4_MISO: now reaches U1.4 (PE5)
- net SPI1_NSS: now reaches U1.49 (PA4)
- net SPI4_MOSI: now reaches U1.5 (PE6)
- net SPI1_SCK: now reaches U1.50 (PA5)
- net SPI1_MISO: now reaches U1.51 (PA6)
- net SPI2_NSS: now reaches U1.85 (PB12)
- net SPI2_MISO: now reaches U1.87 (PB14)
- net SPI2_MOSI: now reaches U1.88 (PB15)
- net Eth.CRS_DV renamed SPI1_MOSI
- net Eth.MDC: no longer names the net of U1.35 (PC1)
- net Eth.MDIO: no longer names the net of U1.43 (PA2)
- net Eth.REFCLKO: no longer names the net of U1.42 (PA1)
- net Eth.RST renamed SPI4_SCK
- net Eth.RXD0: no longer names the net of U1.53 (PC4)
- net Eth.RXD1: no longer names the net of U1.54 (PC5)
- net Eth.RXER: no longer names the net of U1.110 (PG2)
- net Eth.TXD0 renamed BC1
- net Eth.TXD1 renamed SPI2_SCK
- net Eth.TXEN: no longer names the net of U1.155 (PG11)

Commit message: arthur
Connections:
- net led1: now reaches U1.110 (PG2)
- net led2: now reaches U1.111 (PG3)
- net ADS_loadcell: now reaches U1.154 (PG10)
- net ADC_4theromocouple: now reaches U1.155 (PG11)
- net led0: now reaches U1.66 (PG1)
Changed lines of the file:
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@@
+	(wire
+		(pts
+			(xy 116.84 134.62) (xy 121.92 134.62)
+		)
+		(stroke
+			(width 0)
+			(type default)
+		)
+	)
 	(wire
 		(pts
@@
 	(wire
 		(pts
+			(xy 116.84 111.76) (xy 121.92 111.76)
+		)
+		(stroke
+			(width 0)
+			(type default)
+		)
+	)
+	(wire
+		(pts
 			(xy 115.57 172.72) (xy 121.92 172.72)
 		)
@@
 	(wire
 		(pts
+			(xy 116.84 114.3) (xy 121.92 114.3)
+		)
+		(stroke
+			(width 0)
+			(type default)
+		)
+	)
+	(wire
+		(pts
 			(xy 267.97 189.23) (xy 264.16 189.23)
 		)
@@
 	(wire
 		(pts
+			(xy 116.84 132.08) (xy 121.92 132.08)
+		)
+		(stroke
+			(width 0)
+			(type default)
+		)
+	)
+	(wire
+		(pts
 			(xy 160.02 44.45) (xy 160.02 50.8)
 		)
@@
 		(pts
 			(xy 175.26 44.45) (xy 172.72 44.45)
+		)
+		(stroke
+			(width 0)
+			(type default)
+		)
+	)
+	(wire
+		(pts
+			(xy 116.84 109.22) (xy 121.92 109.22)
 		)
 		(stroke
@@
 		)
 	)
+	(hierarchical_label "ADC_4theromocouple"
+		(shape output)
+		(at 116.84 134.62 180)
+		(effects
+			(font
+				(size 1.27 1.27)
+			)
+			(justify right)
+		)
+	)
+	(hierarchical_label "led2"
+		(shape output)
+		(at 116.84 114.3 180)
+		(effects
+			(font
+				(size 1.27 1.27)
+			)
+			(justify right)
+		)
+	)
 	(hierarchical_label "JTCK"
 		(shape input)
@@
 		)
 	)
+	(hierarchical_label "led0"
+		(shape output)
+		(at 116.84 109.22 180)
+		(effects
+			(font
+				(size 1.27 1.27)
+			)
+			(justify right)
+		)
+	)
 	(hierarchical_label "SD.CLK"
 		(shape input)
@@
 		)
 	)
+	(hierarchical_label "ADS_loadcell"
+		(shape output)
+		(at 116.84 132.08 180)
+		(effects
+			(font
+				(size 1.27 1.27)
+			)
+			(justify right)
+		)
+	)
 	(hierarchical_label "SPI1_NSS"
 		(shape input)
@@
 		)
 	)
+	(hierarchical_label "led1"
+		(shape output)
+		(at 116.84 111.76 180)
+		(effects
+			(font
+				(size 1.27 1.27)
+			)
+			(justify right)
+		)
+	)

Commit message: Mis a jour plusieurs circuit et ajouter beaucoup de footprint manquant
Parts:
- removed C14, C15, C16, C17, C18, C2, C3, C33, C4, C5, C8: *, symbol Device:C
- removed C27: 6pF, symbol Device:C
- removed R16, R40: 0, symbol Device:R_US
- removed R27: 100k, symbol Device:R_US
- removed SW1: CK_KMS2xxG, Button_Switch_SMD:SW_SPST_CK_KMS2xxGP, symbol Switch:CK_KMS2xxG
- removed Y1, Y2: Crystal, Crystal:Crystal_SMD_3225-4Pin_3.2x2.5mm, symbol Device:Crystal
- added C48, C66, C67, C68, C69, C70, C71, C72, C73, C74, C75, C76, C77, C78, C88, C90, C92, C93: 100n, Capacitor_SMD:C_0402_1005Metric, symbol Device:C
- added C49, C57: 10u, Capacitor_SMD:C_0402_1005Metric, symbol Device:C
- added C50: *, Capacitor_SMD:C_0402_1005Metric, symbol Device:C
- added C87, C89: 100n, Capacitor_SMD:C_0603_1608Metric_Pad1.08x0.95mm_HandSolder, symbol Device:C
- added C91: 100n, Capacitor_SMD:C_0603_1608Metric, symbol Device:C
- added C94, C95, C96, C97: 1u, Capacitor_SMD:C_0603_1608Metric, symbol Device:C
- added C98: 4.7u, Capacitor_SMD:C_0603_1608Metric, symbol Device:C
- added R20: 10k, Capacitor_SMD:C_0402_1005Metric, symbol Device:R_US
- added R21: 10k, Resistor_SMD:R_0603_1608Metric_Pad0.98x0.95mm_HandSolder, symbol Device:R_US
- added R29: 0, Capacitor_SMD:C_0402_1005Metric, symbol Device:R_US
- added SW3: CK_KMS2xxG, Button_Switch_SMD:SW_SPST_CK_KMS2xxGP, symbol Switch:CK_KMS2xxG
- added Y4: ASV-25.000MHz, Oscillator:Oscillator_SMD_Abracon_ASV-4Pin_7.0x5.1mm, symbol Oscillator:ASV-xxxMHz
- added Y5: ASV-32.768kHz, Oscillator:Oscillator_SMD_Abracon_ASV-4Pin_7.0x5.1mm, symbol Oscillator:ASV-xxxMHz
- C1, C19, C20, C23, C24, C25, C31, C32: footprint (none) -> Capacitor_SMD:C_0603_1608Metric
- C26: value 6pF -> 100n; footprint (none) -> Capacitor_SMD:C_0402_1005Metric
- C34: value * -> 100n; footprint (none) -> Capacitor_SMD:C_0402_1005Metric
- R14: footprint (none) -> Resistor_SMD:R_0603_1608Metric_Pad0.98x0.95mm_HandSolder
- R15: value 0 -> 100k; footprint (none) -> Resistor_SMD:R_0603_1608Metric_Pad0.98x0.95mm_HandSolder
- R39: footprint (none) -> Resistor_SMD:R_0603_1608Metric
Connections:
- net 3V3: now also C34.1, R15.1, C48.1, C49.1, C57.1, C66.1, C67.1, C68.1, C69.1, C70.1, C71.1, C72.1, C73.1, C74.1, C75.1, C76.1, C77.1, C78.1, C87.1, C88.1, C89.1, C90.1, C91.1, C92.1, C93.1, C94.1, C95.1, C96.1, C97.1, C98.1, R20.1, R21.1, Y4.4 (Vdd), Y5.4 (Vdd)
- net GND: now also C26.2, C48.2, C49.2, C50.2, C57.2, C66.2, C67.2, C68.2, C69.2, C70.2, C71.2, C72.2, C73.2, C74.2, C75.2, C76.2, C77.2, C78.2, C87.2, C88.2, C89.2, C90.2, C91.2, C92.2, C93.2, C94.2, C95.2, C96.2, C97.2, C98.2, SW3.1, SW3.SH (B), Y4.2 (GND), Y5.2 (GND); no longer C26.1
- net Clock_32.768kHz: now reaches U1.10 (PC14)
- net Boot: now reaches R14.2, U1.167 (BOOT0)
- net Clock_25MHz: now reaches U1.31 (PH0)
- net Clock_25MHz: no longer R15.2
- net NRST: now reaches U1.33 (NRST)
- net NRST: now also C26.1, R15.2, SW3.2
- net PE13: now reaches U1.75 (PE13)
- net PE14: now reaches U1.76 (PE14)
- net PE15: now reaches U1.77 (PE15)
- removed net Eth.CLKIN: C26.2, R15.1
- net JTCK renamed SWCLK
- net JTDI: no longer names the net of U1.139 (PA15)
- net JTDO renamed SWO
- net JTMS renamed SWDIO
- net NJTRST: no longer names the net of U1.163 (PB4)
- new net: R21.2, Y5.1 (EN)
- new net: R20.2, Y4.1 (EN)
- new net: R29.1, Y4.3 (OUT)
- new net Clock_25Mhz: C50.1, R29.2
- new net Clock_32.768khz: Y5.3 (OUT)
- no-connect marks 5 -> 9
Other:
- note added: "BOOT"
- note added: "DECOUPLING MCU"
- note added: "EXTERNAL OSCILLATOR"
- note added: "RESET"
- note removed: "Découplage"
- moved on the sheet: C1, C19, C20, SW2
